Commit message: Commit 14 [1:04:50]: Still trying to get urdf to work, object isn't showing up on rviz screen.

File: src/urdf_tutorial/urdf/simple-link.urdf (robot description, URDF)
Before this commit: robot materials, 1 links, 0 joints
Links:
- added link world
Joints:
- added joint world_to_base: type fixed, parent world, child base_link, origin xyz=0 0 0 rpy=0 0 0
